File: _autosave-typisttae40v3-pcb.sch (KiCad schematic (older format))
At the start: 1 part

Commit message: end of the night 3:30am [finished part 3]
Parts:
- added C?: 1uF, symbol Device:C_Small
- added C? (x3): 0.1uF, symbol Device:C_Small
- added C?: 10uF, symbol Device:C_Small
- added C? (x2): 22pF, symbol Device:C_Small
- added R? (x2): 10k, symbol Device:R_Small
- added R? (x2): 22, symbol Device:R_Small
- added SW?: SW_Push, symbol Switch:SW_Push
- added Y?: 16MHz, symbol Device:Crystal_GND24_Small
Connections:
- net +5V: now also U?.7 (VBUS), C?.1, C?.1, C?.1, C?.1, R?.1
- net GND: now also C?.2, C?.2, C?.2, C?.2, C?.2, C?.2, C?.2, R?.1, SW?.1, Y?.2, Y?.4
- net at U?.13 (~RESET): now also R?.2, SW?.2
- net at U?.16 (XTAL2): now also C?.1, Y?.3
- net at U?.17 (XTAL1): now also C?.1, Y?.1
- net at U?.3 (D-): now also R?.1
- net at U?.33 (~HWB~/PE2): now also R?.2
- net at U?.4 (D+): now also R?.1
- net at U?.6 (UCAP): now also C?.1
- new net D+: R?.2

Commit message: autosave while pc was in sleep mode
Connections:
- net D-: now reaches R?.2
Other:
- moved on the sheet: R?
Changed lines of the file:
@@
 L Device:R_Small R?
 U 1 1 62EADDC5
-P 5600 2550
-F 0 "R?" V 5404 2550 50  0000 C CNN
-F 1 "22" V 5495 2550 50  0000 C CNN
-F 2 "" H 5600 2550 50  0001 C CNN
-F 3 "~" H 5600 2550 50  0001 C CNN
-	1    5600 2550
+P 6000 2550
+F 0 "R?" V 5804 2550 50  0000 C CNN
+F 1 "22" V 5895 2550 50  0000 C CNN
+F 2 "" H 6000 2550 50  0001 C CNN
+F 3 "~" H 6000 2550 50  0001 C CNN
+	1    6000 2550
 	0    1    1    0
 $EndComp
@@
 	6100 2450 5850 2450
 Wire Wire Line
-	6800 2550 5700 2550
+	6800 2550 6100 2550
 $Comp
 L Device:C_Small C?
@@
 Wire Wire Line
 	6750 1450 6650 1450
-Wire Wire Line
-	5200 2550 5500 2550
 Text GLabel 5850 2450 0    50   Input ~ 0
 D+
+Text GLabel 5850 2550 0    50   Input ~ 0
+D-
+Wire Wire Line
+	5900 2550 5850 2550
 $EndSCHEMATC

Commit message: progress on step six before playing val
Parts:
- added D? (x2): D_Small, symbol Device:D_Small
- added F?: 500mA, symbol Device:Polyfuse_Small
- added MX? (x2): MX-NoLED, symbol MX_Alps_Hybrid:MX-NoLED
- added USB?: Molex-0548190589, symbol random-keyboard-parts:Molex-0548190589
Connections:
- net +5V: now also F?.1
- net D+: now also USB?.3 (D+)
- net D-: now also USB?.4 (D-)
- net GND: now also USB?.1 (GND)
- new net: D?.2 (A), MX?.2 (ROW) (x2)
- new net VCC: F?.2, USB?.5 (VBUS)
Changed lines of the file:
@@
 Wire Wire Line
 	5900 2550 5850 2550
+$Comp
+L random-keyboard-parts:Molex-0548190589 USB?
+U 1 1 62EDE864
+P 9000 1600
+F 0 "USB?" V 9537 1567 60  0000 C CNN
+F 1 "Molex-0548190589" V 9431 1567 60  0000 C CNN
+F 2 "" H 9000 1600 60  0001 C CNN
+F 3 "" H 9000 1600 60  0001 C CNN
+	1    9000 1600
+	0    -1   -1   0
+$EndComp
+$Comp
+L Device:Polyfuse_Small F?
+U 1 1 62EDFB9E
+P 9900 1400
+F 0 "F?" V 9695 1400 50  0000 C CNN
+F 1 "500mA" V 9786 1400 50  0000 C CNN
+F 2 "" H 9950 1200 50  0001 L CNN
+F 3 "~" H 9900 1400 50  0001 C CNN
+	1    9900 1400
+	0    1    1    0
+$EndComp
+Wire Wire Line
+	9300 1400 9600 1400
+$Comp
+L power:+5V #PWR?
+U 1 1 62EE3D21
+P 10400 1400
+F 0 "#PWR?" H 10400 1250 50  0001 C CNN
+F 1 "+5V" H 10415 1573 50  0000 C CNN
+F 2 "" H 10400 1400 50  0001 C CNN
+F 3 "" H 10400 1400 50  0001 C CNN
+	1    10400 1400
+	1    0    0    -1
+$EndComp
+Wire Wire Line
+	10400 1400 10000 1400
+$Comp
+L power:VCC #PWR?
+U 1 1 62EE4CDE
+P 9600 1400
+F 0 "#PWR?" H 9600 1250 50  0001 C CNN
+F 1 "VCC" H 9617 1573 50  0000 C CNN
+F 2 "" H 9600 1400 50  0001 C CNN
+F 3 "" H 9600 1400 50  0001 C CNN
+	1    9600 1400
+	1    0    0    -1
+$EndComp
+Connection ~ 9600 1400
+Wire Wire Line
+	9600 1400 9800 1400
+Text GLabel 9300 1500 2    50   Input ~ 0
+D-
+Text GLabel 9300 1600 2    50   Input ~ 0
+D+
+$Comp
+L power:GND #PWR?
+U 1 1 62EE61B6
+P 9450 1800
+F 0 "#PWR?" H 9450 1550 50  0001 C CNN
+F 1 "GND" H 9455 1627 50  0000 C CNN
+F 2 "" H 9450 1800 50  0001 C CNN
+F 3 "" H 9450 1800 50  0001 C CNN
+	1    9450 1800
+	1    0    0    -1
+$EndComp
+Wire Wire Line
+	9450 1800 9300 1800
+$Comp
+L MX_Alps_Hybrid:MX-NoLED MX?
+U 1 1 62EE7856
+P 8600 2450
+F 0 "MX?" H 8633 2673 60  0000 C CNN
+F 1 "MX-NoLED" H 8633 2599 20  0000 C CNN
+F 2 "" H 7975 2425 60  0001 C CNN
+F 3 "" H 7975 2425 60  0001 C CNN
+	1    8600 2450
+	1    0    0    -1
+$EndComp
+$Comp
+L Device:D_Small D?
+U 1 1 62EEAB86
+P 8400 2700
+F 0 "D?" V 8446 2632 50  0000 R CNN
+F 1 "D_Small" V 8355 2632 50  0000 R CNN
+F 2 "" V 8400 2700 50  0001 C CNN
+F 3 "~" V 8400 2700 50  0001 C CNN
+	1    8400 2700
+	0    -1   -1   0
+$EndComp
+Wire Wire Line
+	8550 2600 8400 2600
+$Comp
+L MX_Alps_Hybrid:MX-NoLED MX?
+U 1 1 62EED4A2
+P 9200 2450
+F 0 "MX?" H 9233 2673 60  0000 C CNN
+F 1 "MX-NoLED" H 9233 2599 20  0000 C CNN
+F 2 "" H 8575 2425 60  0001 C CNN
+F 3 "" H 8575 2425 60  0001 C CNN
+	1    9200 2450
+	1    0    0    -1
+$EndComp
+$Comp
+L Device:D_Small D?
+U 1 1 62EF6235
+P 9000 2700
+F 0 "D?" V 9046 2632 50  0000 R CNN
+F 1 "D_Small" V 8955 2632 50  0000 R CNN
+F 2 "" V 9000 2700 50  0001 C CNN
+F 3 "~" V 9000 2700 50  0001 C CNN
+	1    9000 2700
+	0    -1   -1   0
+$EndComp
+Wire Wire Line
+	9000 2600 9150 2600
 $EndSCHEMATC

Commit message: PCB Guide Part 4 Complete!
Parts:
- added D2, D3: SOD-123, symbol Device:D_Small
- added MX2, MX3: MX-NoLED, symbol MX_Alps_Hybrid:MX-NoLED
- C1, C2, C3, C4, C5, C6, C7: renamed from C?; footprint (none) -> Capacitor_SMD:C_0805_2012Metric
- D1, D4: renamed from D?; value D_Small -> SOD-123
- gave numbers to parts that had none: 11
Connections:
- net COL1: now reaches MX4.1 (COL)
- net COL1: now also MX3.1 (COL)
- net ROW1: now reaches D4.1 (K)
- net ROW1: now also D2.1 (K)
- net COL0: now reaches MX1.1 (COL)
- net COL0: now also MX2.1 (COL)
- net ROW0: now reaches D1.1 (K)
- net ROW0: now also D3.1 (K)
- new net: D2.2 (A), MX2.2 (ROW)
- new net: D3.2 (A), MX3.2 (ROW)
Other:
- moved on the sheet: D1, D4, MX1, MX4
